Commit message: added torque sensors in Gazebo sim

File: light_ws/src/trikey/urdf/trikey_light.urdf.xacro (robot description, xacro)
@@ -24,104 +24,118 @@
         </collision>
     </link>
-    <!-- Three Shaft and Wheel Assemblies -->
-    <xacro:macro name="shaft_wheel" params="id x y rpy">
-        <link name="shaft_link_${id}">
-            <inertial>
-                <origin xyz="0.0 1.2 1.0" rpy="1.5708 0.0 0.0"/>
-                <mass value="1.0"/>
-                <inertia ixx="1.333" ixy="0.0" ixz="0.0" iyy="0.0" iyz="0.0" izz="1.333"/>
-            </inertial>
-            <visual>
-                <origin xyz="0.0 1.2 1.0" rpy="1.5708 0.0 0.0"/>
-                <geometry>
-                    <cylinder radius="0.5" length="2"/>
-                </geometry>
-                <material name="red">
-                    <color rgba="1.0 0.0 0.0 1.0"/>
-                </material>
-            </visual>
-            <collision>
-                <origin xyz="0.0 1.2 1.0" rpy="1.5708 0.0 0.0"/>
-                <geometry>
-                    <cylinder radius="0.5" length="2"/>
-                </geometry>
-            </collision>
-        </link>
-        <joint name="base_joint_${id}" type="fixed">
-            <origin xyz="${x} ${y} 0.0" rpy="0.0 0.0 ${rpy}"/>
-            <parent link="center_link"/>
-            <child link="shaft_link_${id}"/>
-        </joint>
-        <link name="wheel_link_${id}">
-            <inertial>
-                <origin xyz="0.0 0.0 0.0" rpy="0.0 0.0 0.0"/>
-                <mass value="0.5"/>
-                <inertia ixx="0.5" ixy="0.0" ixz="0.0" iyy="0.25" iyz="0.0" izz="0.5"/>
-            </inertial>
-            <visual>
-                <origin xyz="0.0 0.0 -0.2" rpy="0.0 0.0 0.0"/>
-                <geometry>
-                    <cylinder radius="1.0" length="0.3"/>
-                </geometry>
-                <material name="black">
-                    <color rgba="0.0 0.0 0.0 1.0"/>
-                </material>
-            </visual>
-            <surface>
-                <friction>
-                <ode>
-                    <mu>100</mu>
-                    <mu2>100</mu2>
-                </ode>
-                </friction>
-                <contact>
-                <ode>
-                    <min_depth>0.003</min_depth>
-                </ode>
+  <xacro:macro name="shaft_wheel" params="id x y rpy">
+    <!-- Shaft -->
+    <link name="shaft_link_${id}">
+      <inertial>
+        <origin xyz="0.0 1.2 1.0" rpy="1.5708 0.0 0.0"/>
+        <mass value="1.0"/>
+        <inertia ixx="1.333" ixy="0.0" ixz="0.0" iyy="0.0" iyz="0.0" izz="1.333"/>
+      </inertial>
+      <visual>
+        <origin xyz="0.0 1.2 1.0" rpy="1.5708 0.0 0.0"/>
+        <geometry>
+          <cylinder radius="0.5" length="2"/>
+        </geometry>
+        <material name="red">
+          <color rgba="1.0 0.0 0.0 1.0"/>
+        </material>
+      </visual>
+      <collision>
+        <origin xyz="0.0 1.2 1.0" rpy="1.5708 0.0 0.0"/>
+        <geometry>
+          <cylinder radius="0.5" length="2"/>
+        </geometry>
+      </collision>
+    </link>
+    <!-- Fixed joint attaching the shaft to the robot base -->
+    <joint name="base_joint_${id}" type="fixed">
+      <origin xyz="${x} ${y} 0.0" rpy="0.0 0.0 ${rpy}"/>
+      <parent link="center_link"/>
+      <child link="shaft_link_${id}"/>
+    </joint>
+    <!-- Wheel Link -->
+    <link name="wheel_link_${id}">
+      <inertial>
+        <origin xyz="0.0 0.0 0.0" rpy="0.0 0.0 0.0"/>
+        <mass value="0.5"/>
+        <inertia ixx="0.5" ixy="0.0" ixz="0.0" iyy="0.25" iyz="0.0" izz="0.5"/>
+      </inertial>
+      <visual>
+        <origin xyz="0.0 0.0 -0.2" rpy="0.0 0.0 0.0"/>
+        <geometry>
+          <cylinder radius="1.0" length="0.3"/>
+        </geometry>
+        <material name="black">
+          <color rgba="0.0 0.0 0.0 1.0"/>
+        </material>
+      </visual>
+      <surface>
+        <friction>
+          <ode>
+            <mu>100</mu>
+            <mu2>100</mu2>
+          </ode>
+        </friction>
+        <contact>
+          <ode>
+            <min_depth>0.003</min_depth>
+          </ode>
         </contact>
-            </surface>
-            <collision>
-                <origin xyz="0.0 0.0 0.0" rpy="0.0 0.0 0.0"/>
-                <geometry>
-                    <cylinder radius="1.0" length="0.3"/>
-                </geometry>
-            </collision>
-        </link>
-        <joint name="wheel_joint_${id}" type="continuous">
-            <origin xyz="0.0 2.0 1.0" rpy="1.57 0.0 0.0"/>
-            <parent link="shaft_link_${id}"/>
-            <child link="wheel_link_${id}"/>
-            <axis xyz="0.0 0.0 1.0"/>
-            <limit effort="10.0" velocity="5.0"/>
-        </joint>
-        <transmission name="wheel_joint_transmission_${id}">
-            <type>transmission_interface/SimpleTransmission</type>
-            <joint name="wheel_joint_${id}">
-                <hardwareInterface>hardware_interface/EffortJointInterface</hardwareInterface>
-            </joint>
-            <actuator name="wheel_motor_${id}">
-                <hardwareInterface>hardware_interface/EffortJointInterface</hardwareInterface>
-                <mechanicalReduction>1</mechanicalReduction>
-            </actuator>
-        </transmission>
-    </xacro:macro>
-    <!-- Instantiate three shaft-wheel assemblies at 120-degree intervals -->
-    <!-- <xacro:shaft_wheel id="1" x="1.2" y="0.0" rpy="0.0"/>
-    <xacro:shaft_wheel id="2" x="-0.6" y="1.039" rpy="2.094"/>
-    <xacro:shaft_wheel id="3" x="-0.6" y="-1.039" rpy="-2.094"/> -->
-<!--
-    <xacro:shaft_wheel id="1" x="1" y="0.0" rpy="1.5708"/>
-    <xacro:shaft_wheel id="2" x="-0.5" y="0.8660254038" rpy="3.66519"/>
-    <xacro:shaft_wheel id="3" x="-0.5" y="-0.8660254038" rpy="5.75959"/> -->
-    <xacro:property name="r" value="-1"/>
+      </surface>
+      <collision>
+        <origin xyz="0.0 0.0 0.0" rpy="0.0 0.0 0.0"/>
+        <geometry>
+          <cylinder radius="1.0" length="0.3"/>
+        </geometry>
+      </collision>
+    </link>
+    <!-- Continuous joint connecting the shaft to the wheel, with embedded FT sensor -->
+    <joint name="wheel_joint_${id}" type="continuous">
+      <origin xyz="0.0 2.0 1.0" rpy="1.57 0.0 0.0"/>
+      <parent link="shaft_link_${id}"/>
+      <child link="wheel_link_${id}"/>
+      <axis xyz="0.0 0.0 1.0"/>
+      <limit effort="10.0" velocity="5.0"/>
+    <provideFeedback>true</provideFeedback>
+      <physics>
+            <provideFeedback>true</provideFeedback>
+        </physics>
+      <gazebo>
+            <physics>
+            <provideFeedback>true</provideFeedback>
+            </physics>
+            <provideFeedback>true</provideFeedback>
+        <sensor type="force_torque" name="ft_sensor_wheel_${id}">
+          <always_on>true</always_on>
+          <update_rate>100</update_rate>
+          <force_torque>
+            <frame>child</frame>
+          </force_torque>
+        </sensor>
+      </gazebo>
+    </joint>
+    <!-- Transmission referencing the continuous joint -->
+    <transmission name="wheel_joint_transmission_${id}">
+      <type>transmission_interface/SimpleTransmission</type>
+      <joint name="wheel_joint_${id}">
+        <hardwareInterface>hardware_interface/EffortJointInterface</hardwareInterface>
+      </joint>
+      <actuator name="wheel_motor_${id}">
+        <hardwareInterface>hardware_interface/EffortJointInterface</hardwareInterface>
+        <mechanicalReduction>1</mechanicalReduction>
+      </actuator>
+    </transmission>
+    <gazebo reference="wheel_joint_${id}">
+        <provideFeedback>true</provideFeedback>
+    </gazebo>
+  </xacro:macro>
+  <!-- Instantiate three shaft/wheel assemblies at 0°, +120°, -120° -->
+  <xacro:property name="r" value="-1"/>
   <!-- Angles in radians -->
-  <!-- 0°, 120°, and -120° in radians -->
   <xacro:property name="theta1" value="0.0"/>
   <xacro:property name="theta2" value="2.0943951"/>    <!-- 120 deg -->
   <xacro:property name="theta3" value="-2.0943951"/>   <!-- -120 deg -->
-  <!-- If you need to add 90° (pi/2 = 1.5708) to each rotation: -->
+  <!-- Additional rotation if needed -->
   <xacro:property name="rotate90" value="1.5708"/>
-      <!-- Instantiate three shafts/wheels at 0°, +120°, -120° -->
-  <!-- We add +90° (rotate90) to each RPY if needed. -->
   <xacro:shaft_wheel
       id="1"
@@ -142,8 +156,46 @@
       rpy="${theta3 + rotate90}"
   />
-    <gazebo>
-        <plugin name="gazebo_ros_control" filename="libgazebo_ros_control.so">
-            <robotNamespace>/trikey_light</robotNamespace>
-        </plugin>
-    </gazebo>
+  <gazebo>
+      <provideFeedback>true</provideFeedback>
+    <plugin name="gazebo_ros_control" filename="libgazebo_ros_control.so">
+      <robotNamespace>/trikey_light</robotNamespace>
+    </plugin>
+    <!-- ros-noetic-gazebo-plugins -->
+    <!-- FT sensor plugin for wheel 1 -->
+    <plugin name="ft_sensor_plugin_1" filename="libgazebo_ros_ft_sensor.so">
+      <ros>
+        <namespace>/trikey_light</namespace>
+        <remapping>~/ft : ft_sensor_1</remapping>
+      </ros>
+      <update_rate>100</update_rate>
+      <bodyName>wheel_link_1</bodyName>
+      <jointName>wheel_joint_1</jointName>
+      <sensorName>ft_sensor_wheel_1</sensorName>
+      <topicName>ft_sensor_1_topic</topicName>
+    </plugin>
+    <!-- FT sensor plugin for wheel 2 -->
+    <plugin name="ft_sensor_plugin_2" filename="libgazebo_ros_ft_sensor.so">
+      <ros>
+        <namespace>/trikey_light</namespace>
+        <remapping>~/ft : ft_sensor_2</remapping>
+      </ros>
+      <update_rate>100</update_rate>
+      <bodyName>wheel_link_2</bodyName>
+      <jointName>wheel_joint_2</jointName>
+      <sensorName>ft_sensor_wheel_2</sensorName>
+      <topicName>ft_sensor_2_topic</topicName>
+    </plugin>
+    <!-- FT sensor plugin for wheel 3 -->
+    <plugin name="ft_sensor_plugin_3" filename="libgazebo_ros_ft_sensor.so">
+      <ros>
+        <namespace>/trikey_light</namespace>
+        <remapping>~/ft : ft_sensor_3</remapping>
+      </ros>
+      <update_rate>100</update_rate>
+      <bodyName>wheel_link_3</bodyName>
+      <jointName>wheel_joint_3</jointName>
+      <sensorName>ft_sensor_wheel_3</sensorName>
+      <topicName>ft_sensor_3_topic</topicName>
+    </plugin>
+  </gazebo>
 </robot>

Commit message: modified:   light_ws/src/trikey/config/joint_controller.yaml 	modified:   light_ws/src/trikey/launch/trikey_gazebo.launch 	modified:   light_ws/src/trikey/rviz/rviz.rviz 	modified:   light_ws/src/trikey/trikey_jacobian.py 	modified:   light_ws/src/trikey/urdf/trikey_light.urdf.xacro

File: light_ws/src/trikey/urdf/trikey_light.urdf.xacro (robot description, xacro)
@@ -73,11 +73,14 @@
         <friction>
           <ode>
-            <mu>100000</mu>
-            <mu2>100000</mu2>
+            <mu>10</mu>
+            <mu2>0.1</mu2>
           </ode>
         </friction>
         <contact>
           <ode>
-            <min_depth>0.005</min_depth>
+              <kp>1e5</kp>
+              <kd>1e3</kd>
+              <max_vel>2</max_vel>
+              <min_depth>0.001</min_depth>
           </ode>
         </contact>
@@ -96,5 +99,5 @@
       <child link="wheel_link_${id}"/>
       <axis xyz="0.0 0.0 1.0"/>
-      <limit effort="10.0" velocity="5.0"/>
+      <limit effort="100.0" velocity="10.0"/>
     <provideFeedback>true</provideFeedback>
       <physics>
@@ -108,5 +111,5 @@
         <sensor type="force_torque" name="ft_sensor_wheel_${id}">
           <always_on>true</always_on>
-          <update_rate>100</update_rate>
+          <update_rate>1000</update_rate>
           <force_torque>
             <frame>child</frame>
@@ -120,8 +123,8 @@
       <type>transmission_interface/SimpleTransmission</type>
       <joint name="wheel_joint_${id}">
-        <hardwareInterface>hardware_interface/EffortJointInterface</hardwareInterface>
+        <hardwareInterface>hardware_interface/VelocityJointInterface</hardwareInterface>
       </joint>
       <actuator name="wheel_motor_${id}">
-        <hardwareInterface>hardware_interface/EffortJointInterface</hardwareInterface>
+        <hardwareInterface>hardware_interface/VelocityJointInterface</hardwareInterface>
         <mechanicalReduction>1</mechanicalReduction>
       </actuator>
@@ -157,4 +160,94 @@
       rpy="${theta3 + rotate90}"
   />
+  <!-- Roll Cage Beam between wheel 1 and wheel 2 -->
+  <link name="rollcage_12">
+    <inertial>
+      <origin xyz="0 0 0" rpy="0 0 0"/>
+      <mass value="0.1"/>
+      <inertia ixx="0.0001" ixy="0.0" ixz="0.0"
+               iyy="0.0001" iyz="0.0" izz="0.0001"/>
+    </inertial>
+    <visual>
+      <!-- Midpoint at (-0.25, -0.433, 0), rotated so the cylinder lies along the beam -->
+      <origin xyz="-0.85 -1.4722 1" rpy="0 -1.5708 -0.5236"/>
+      <geometry>
+               <cylinder radius="0.3" length="5"/>
+      </geometry>
+      <material name="silver">
+        <color rgba="0.7 0.7 0.7 1.0"/>
+      </material>
+    </visual>
+    <collision>
+      <origin xyz="-0.85 -1.4722 1" rpy="0 -1.5708 -0.5236"/>
+      <geometry>
+                <cylinder radius="0.3" length="5"/>
+      </geometry>
+    </collision>
+  </link>
+  <joint name="rollcage_joint_12" type="fixed">
+    <origin xyz="0 0 0" rpy="0 0 0"/>
+    <parent link="center_link"/>
+    <child link="rollcage_12"/>
+  </joint>
+  <!-- Roll Cage Beam between wheel 2 and wheel 3 -->
+  <link name="rollcage_23">
+    <inertial>
+      <origin xyz="0 0 0" rpy="0 0 0"/>
+      <mass value="0.1"/>
+      <inertia ixx="0.0001" ixy="0.0" ixz="0.0"
+               iyy="0.0001" iyz="0.0" izz="0.0001"/>
+    </inertial>
+    <visual>
+      <!-- Midpoint at (0.5, 0, 0); beam angle ψ = +1.5708 rad -->
+      <origin xyz="1.7 0 1" rpy="0 -1.5708 1.5708"/>
+      <geometry>
+        <cylinder radius="0.3" length="5"/>
+      </geometry>
+      <material name="silver">
+        <color rgba="0.7 0.7 0.7 1.0"/>
+      </material>
+    </visual>
+    <collision>
+      <origin xyz="1.7 0 1" rpy="0 -1.5708 1.5708"/>
+      <geometry>
+        <cylinder radius="0.3" length="5"/>
+      </geometry>
+    </collision>
+  </link>
+  <joint name="rollcage_joint_23" type="fixed">
+    <origin xyz="0 0 0" rpy="0 0 0"/>
+    <parent link="center_link"/>
+    <child link="rollcage_23"/>
+  </joint>
+  <!-- Roll Cage Beam between wheel 3 and wheel 1 -->
+  <link name="rollcage_31">
+    <inertial>
+      <origin xyz="0 0 0" rpy="0 0 0"/>
+      <mass value="0.1"/>
+      <inertia ixx="0.0001" ixy="0.0" ixz="0.0"
+               iyy="0.0001" iyz="0.0" izz="0.0001"/>
+    </inertial>
+    <visual>
+      <!-- Midpoint at (-0.25, 0.433, 0); beam angle ψ = -2.61799 rad -->
+      <origin xyz="-0.85 1.4722 1" rpy="0 -1.5708 -2.61799"/>
+      <geometry>
+                <cylinder radius="0.3" length="5"/>
+      </geometry>
+      <material name="silver">
+        <color rgba="0.7 0.7 0.7 1.0"/>
+      </material>
+    </visual>
+    <collision>
+      <origin xyz="-0.85 1.4722 1" rpy="0 -1.5708 -2.61799"/>
+      <geometry>
+                <cylinder radius="0.3" length="5"/>
+      </geometry>
+    </collision>
+  </link>
+  <joint name="rollcage_joint_31" type="fixed">
+    <origin xyz="0 0 0" rpy="0 0 0"/>
+    <parent link="center_link"/>
+    <child link="rollcage_31"/>
+  </joint>
   <gazebo>
       <provideFeedback>true</provideFeedback>
@@ -183,5 +276,5 @@
         <remapping>~/ft : ft_sensor_2</remapping>
       </ros>
-      <update_rate>100</update_rate>
+      <update_rate>1000</update_rate>
       <frame>child</frame>
                   <measure_direction>child_to_parent</measure_direction>

Commit message: Increased RollCage

File: light_ws/src/trikey/urdf/trikey_light.urdf.xacro (robot description, xacro)
@@ -170,7 +170,7 @@
     <visual>
       <!-- Midpoint at (-0.25, -0.433, 0), rotated so the cylinder lies along the beam -->
-      <origin xyz="-0.85 -1.4722 1" rpy="0 -1.5708 -0.5236"/>
-      <geometry>
-               <cylinder radius="0.3" length="5"/>
+      <origin xyz="-1.615 -2.79718 1" rpy="0 -1.5708 -0.5236"/>
+      <geometry>
+               <cylinder radius="0.3" length="7"/>
       </geometry>
       <material name="silver">
@@ -179,7 +179,7 @@
     </visual>
     <collision>
-      <origin xyz="-0.85 -1.4722 1" rpy="0 -1.5708 -0.5236"/>
-      <geometry>
-                <cylinder radius="0.3" length="5"/>
+      <origin xyz="-1.615 -2.79718 1" rpy="0 -1.5708 -0.5236"/>
+      <geometry>
+                <cylinder radius="0.3" length="7"/>
       </geometry>
     </collision>
@@ -200,7 +200,7 @@
     <visual>
       <!-- Midpoint at (0.5, 0, 0); beam angle ψ = +1.5708 rad -->
-      <origin xyz="1.7 0 1" rpy="0 -1.5708 1.5708"/>
-      <geometry>
-        <cylinder radius="0.3" length="5"/>
+      <origin xyz="3.23 0 1" rpy="0 -1.5708 1.5708"/>
+      <geometry>
+        <cylinder radius="0.3" length="7"/>
       </geometry>
       <material name="silver">
@@ -209,7 +209,7 @@
     </visual>
     <collision>
-      <origin xyz="1.7 0 1" rpy="0 -1.5708 1.5708"/>
-      <geometry>
-        <cylinder radius="0.3" length="5"/>
+      <origin xyz="3.23 0 1" rpy="0 -1.5708 1.5708"/>
+      <geometry>
+        <cylinder radius="0.3" length="7"/>
       </geometry>
     </collision>
@@ -230,7 +230,7 @@
     <visual>
       <!-- Midpoint at (-0.25, 0.433, 0); beam angle ψ = -2.61799 rad -->
-      <origin xyz="-0.85 1.4722 1" rpy="0 -1.5708 -2.61799"/>
-      <geometry>
-                <cylinder radius="0.3" length="5"/>
+      <origin xyz="-1.615 2.79718 1" rpy="0 -1.5708 -2.61799"/>
+      <geometry>
+                <cylinder radius="0.3" length="7"/>
       </geometry>
       <material name="silver">
@@ -239,7 +239,7 @@
     </visual>
     <collision>
-      <origin xyz="-0.85 1.4722 1" rpy="0 -1.5708 -2.61799"/>
-      <geometry>
-                <cylinder radius="0.3" length="5"/>
+      <origin xyz="-1.615 2.79718 1" rpy="0 -1.5708 -2.61799"/>
+      <geometry>
+                <cylinder radius="0.3" length="7"/>
       </geometry>
     </collision>

Commit message: modified:   light_ws/src/trikey/urdf/trikey_light.urdf.xacro

File: light_ws/src/trikey/urdf/trikey_light.urdf.xacro (robot description, xacro)
@@ -9,5 +9,5 @@
         </inertial> -->
         <visual>
-            <origin xyz="0.0 0.0 1.0" rpy="0.0 0.0 0.0"/>
+            <origin xyz="0.0 0.0 1" rpy="0.0 0.0 0.0"/>
             <geometry>
                 <cylinder radius="0.6" length="0.5"/>
@@ -18,5 +18,5 @@
         </visual>
         <collision>
-            <origin xyz="0.0 0.0 1.0" rpy="0.0 0.0 0.0"/>
+            <origin xyz="0.0 0.0 1.2" rpy="0.0 0.0 0.0"/>
             <geometry>
                 <cylinder radius="0.6" length="0.5"/>
@@ -24,4 +24,33 @@
         </collision>
     </link>
+<!-- Body Link (Raises Center of Mass)-->
+    <link name="body_link">
+        <inertial>
+            <origin xyz="0.0 0.0 0" rpy="0.0 0.0 0.0"/>
+            <mass value="20"/>
+            <inertia ixx="2.0" ixy="0.0" ixz="0.0" iyy="2.0" iyz="0.0" izz="2.0"/>
+        </inertial>
+        <visual>
+            <origin xyz="0.0 0.0 0" rpy="0.0 0.0 0.0"/>
+            <geometry>
+                <cylinder radius="0.6" length="0.5"/>
+            </geometry>
+            <material name="gray">
+                <color rgba="0.5 0.5 0.5 1.0"/>
+            </material>
+        </visual>
+        <collision>
+            <origin xyz="0.0 0.0 0" rpy="0.0 0.0 0.0"/>
+            <geometry>
+                <cylinder radius="0.6" length="0.5"/>
+            </geometry>
+        </collision>
+    </link>
+<!-- Body to Center Joint -->
+<joint name="center_joint" type="fixed">
+    <origin xyz="0 0 0.5" rpy="0 0 0"/>
+    <child link="body_link"/>
+    <parent link="center_link"/>
+</joint>
   <xacro:macro name="shaft_wheel" params="id x y rpy">
     <!-- Shaft -->
@@ -29,5 +58,5 @@
       <inertial>
         <origin xyz="0.0 1.2 1.0" rpy="1.5708 0.0 0.0"/>
-        <mass value="1.0"/>
+        <mass value="5"/>
         <inertia ixx="1.333" ixy="0.0" ixz="0.0" iyy="0.0" iyz="0.0" izz="1.333"/>
       </inertial>
@@ -50,5 +79,5 @@
     <!-- Fixed joint attaching the shaft to the robot base -->
     <joint name="base_joint_${id}" type="fixed">
-      <origin xyz="${x} ${y} 0.0" rpy="0.0 0.0 ${rpy}"/>
+      <origin xyz="${x} ${y} -0.5" rpy="0.0 0.0 ${rpy}"/>
       <parent link="center_link"/>
       <child link="shaft_link_${id}"/>
@@ -57,7 +86,7 @@
     <link name="wheel_link_${id}">
       <inertial>
-        <origin xyz="0.0 0.0 0.0" rpy="0.0 0.0 0.0"/>
-        <mass value="0.5"/>
-        <inertia ixx="0.5" ixy="0.0" ixz="0.0" iyy="0.25" iyz="0.0" izz="0.5"/>
+        <origin xyz="0.0 0.0 -0.2" rpy="0.0 0.0 0.0"/>
+        <mass value="2"/>
+        <inertia ixx="0.25" ixy="0.0" ixz="0.0" iyy="0.25" iyz="0.0" izz="0.5"/>
       </inertial>
       <visual>
@@ -82,10 +111,10 @@
               <kd>1e3</kd>
               <max_vel>2</max_vel>
-              <min_depth>0.001</min_depth>
+              <min_depth>0.003</min_depth>
           </ode>
         </contact>
       </surface>
       <collision>
-        <origin xyz="0.0 0.0 0.0" rpy="0.0 0.0 0.0"/>
+        <origin xyz="0.0 0.0 -0.2" rpy="0.0 0.0 0.0"/>
         <geometry>
           <cylinder radius="1.0" length="0.3"/>
@@ -99,5 +128,5 @@
       <child link="wheel_link_${id}"/>
       <axis xyz="0.0 0.0 1.0"/>
-      <limit effort="100.0" velocity="10.0"/>
+      <limit effort="500.0" velocity="10.0"/>
     <provideFeedback>true</provideFeedback>
       <physics>
