Commit message: Changed model configuration

File: light_ws/src/trikey/urdf/trikey_light.urdf.xacro (robot description, xacro)
@@ -2,5 +2,5 @@
 <robot xmlns:xacro="http://www.ros.org/wiki/xacro"  name="trikey_light">
    <!-- Central Body -->
-    <link name="center_link">
+    <link name="base_link">
         <!-- <inertial>
             <origin xyz="0.0 0.0 1.0" rpy="0.0 0.0 0.0"/>
@@ -51,5 +51,5 @@
     <origin xyz="0 0 0.5" rpy="0 0 0"/>
     <child link="body_link"/>
-    <parent link="center_link"/>
+    <parent link="base_link"/>
 </joint>
   <xacro:macro name="shaft_wheel" params="id x y rpy">
@@ -80,5 +80,5 @@
     <joint name="base_joint_${id}" type="fixed">
       <origin xyz="${x} ${y} -0.5" rpy="0.0 0.0 ${rpy}"/>
-      <parent link="center_link"/>
+      <parent link="base_link"/>
       <child link="shaft_link_${id}"/>
     </joint>
@@ -128,5 +128,5 @@
       <child link="wheel_link_${id}"/>
       <axis xyz="0.0 0.0 1.0"/>
-      <limit effort="500.0" velocity="10.0"/>
+      <limit effort="300.0" velocity="10.0"/>
     <provideFeedback>true</provideFeedback>
       <physics>
@@ -189,4 +189,52 @@
       rpy="${theta3 + rotate90}"
   />
+  <!-- Macro to add a cover bar for a wheel -->
+<xacro:macro name="wheel_cover_bar" params="id pos_x pos_y pos_z rpy_x rpy_y rpy_z length">
+  <link name="wheel_cover_${id}">
+    <inertial>
+      <origin xyz="0 0 0" rpy="0 0 0"/>
+      <mass value="0.05"/>
+      <inertia ixx="0.001" ixy="0.0" ixz="0.0" iyy="0.001" iyz="0.0" izz="0.001"/>
+    </inertial>
+    <visual>
+      <!-- The cylinder represents the bar cover. Its radius matches the roll cage (0.3) -->
+      <origin xyz="0 0 0" rpy="0 0 0"/>
+      <geometry>
+        <cylinder radius="0.3" length="${length}"/>
+      </geometry>
+      <material name="cover_material">
+        <color rgba="0.7 0.7 0.7 1.0"/>
+      </material>
+    </visual>
+    <collision>
+      <origin xyz="0 0 0" rpy="0 0 0"/>
+      <geometry>
+        <cylinder radius="0.3" length="${length}"/>
+      </geometry>
+    </collision>
+  </link>
+  <joint name="wheel_cover_joint_${id}" type="fixed">
+    <origin xyz="${pos_x} ${pos_y} ${pos_z}" rpy="${rpy_x} ${rpy_y} ${rpy_z}"/>
+    <parent link="base_link"/>
+    <child link="wheel_cover_${id}"/>
+  </joint>
+</xacro:macro>
+<xacro:wheel_cover_bar
+    id="1"
+    pos_x="-4.4" pos_y="0" pos_z="1"
+    rpy_x="0" rpy_y="1.5708" rpy_z="1.5708"
+    length="1.65"/>
+<!-- Cover for Wheel 2 (located at (0.5,-0.866)) -->
+<xacro:wheel_cover_bar
+    id="2"
+    pos_x="2.2" pos_y="-3.81" pos_z="1"
+    rpy_x="0" rpy_y="1.5708" rpy_z="-2.61799"
+    length="1.65"/>
+<!-- Cover bar for Wheel 3 (connecting rollcage_23 and rollcage_31) -->
+<xacro:wheel_cover_bar
+    id="3"
+    pos_x="2.2" pos_y="3.81" pos_z="1"
+    rpy_x="0" rpy_y="1.5708" rpy_z="2.61799"
+    length="1.65"/>
   <!-- Roll Cage Beam between wheel 1 and wheel 2 -->
   <link name="rollcage_12">
@@ -201,5 +249,5 @@
       <origin xyz="-1.615 -2.79718 1" rpy="0 -1.5708 -0.5236"/>
       <geometry>
-               <cylinder radius="0.3" length="7"/>
+               <cylinder radius="0.3" length="6.7"/>
       </geometry>
       <material name="silver">
@@ -210,5 +258,5 @@
       <origin xyz="-1.615 -2.79718 1" rpy="0 -1.5708 -0.5236"/>
       <geometry>
-                <cylinder radius="0.3" length="7"/>
+                <cylinder radius="0.3" length="6.7"/>
       </geometry>
     </collision>
@@ -216,5 +264,5 @@
   <joint name="rollcage_joint_12" type="fixed">
     <origin xyz="0 0 0" rpy="0 0 0"/>
-    <parent link="center_link"/>
+    <parent link="base_link"/>
     <child link="rollcage_12"/>
   </joint>
@@ -231,5 +279,5 @@
       <origin xyz="3.23 0 1" rpy="0 -1.5708 1.5708"/>
       <geometry>
-        <cylinder radius="0.3" length="7"/>
+        <cylinder radius="0.3" length="6.7"/>
       </geometry>
       <material name="silver">
@@ -240,5 +288,5 @@
       <origin xyz="3.23 0 1" rpy="0 -1.5708 1.5708"/>
       <geometry>
-        <cylinder radius="0.3" length="7"/>
+        <cylinder radius="0.3" length="6.5"/>
       </geometry>
     </collision>
@@ -246,5 +294,5 @@
   <joint name="rollcage_joint_23" type="fixed">
     <origin xyz="0 0 0" rpy="0 0 0"/>
-    <parent link="center_link"/>
+    <parent link="base_link"/>
     <child link="rollcage_23"/>
   </joint>
@@ -261,5 +309,5 @@
       <origin xyz="-1.615 2.79718 1" rpy="0 -1.5708 -2.61799"/>
       <geometry>
-                <cylinder radius="0.3" length="7"/>
+                <cylinder radius="0.3" length="6.7"/>
       </geometry>
       <material name="silver">
@@ -270,5 +318,5 @@
       <origin xyz="-1.615 2.79718 1" rpy="0 -1.5708 -2.61799"/>
       <geometry>
-                <cylinder radius="0.3" length="7"/>
+                <cylinder radius="0.3" length="6.7"/>
       </geometry>
     </collision>
@@ -276,5 +324,5 @@
   <joint name="rollcage_joint_31" type="fixed">
     <origin xyz="0 0 0" rpy="0 0 0"/>
-    <parent link="center_link"/>
+    <parent link="base_link"/>
     <child link="rollcage_31"/>
   </joint>

Commit message: modified:   light_ws/src/trikey/config/robot.rviz 	modified:   light_ws/src/trikey/urdf/trikey_light.urdf.xacro

File: light_ws/src/trikey/urdf/trikey_light.urdf.xacro (robot description, xacro)
@@ -194,6 +194,6 @@
     <inertial>
       <origin xyz="0 0 0" rpy="0 0 0"/>
-      <mass value="0.05"/>
-      <inertia ixx="0.001" ixy="0.0" ixz="0.0" iyy="0.001" iyz="0.0" izz="0.001"/>
+      <mass value="0.1"/>
+      <inertia ixx="0.0001" ixy="0.0" ixz="0.0" iyy="0.0001" iyz="0.0" izz="0.0001"/>
     </inertial>
     <visual>
@@ -339,5 +339,6 @@
         <remapping>~/ft : ft_sensor_1</remapping>
       </ros>
-      <update_rate>100</update_rate>
+      <always_on>true</always_on>
+      <update_rate>1000</update_rate>
             <frame>child</frame>
             <measure_direction>child_to_parent</measure_direction>
@@ -353,4 +354,5 @@
         <remapping>~/ft : ft_sensor_2</remapping>
       </ros>
+      <always_on>true</always_on>
       <update_rate>1000</update_rate>
       <frame>child</frame>
@@ -367,5 +369,6 @@
         <remapping>~/ft : ft_sensor_3</remapping>
       </ros>
-      <update_rate>100</update_rate>
+      <always_on>true</always_on>
+      <update_rate>1000</update_rate>
             <frame>child</frame>
             <measure_direction>child_to_parent</measure_direction>

Commit message: modified:   light_ws/src/trikey/config/joint_controller.yaml 	modified:   light_ws/src/trikey/config/robot.rviz 	modified:   light_ws/src/trikey/launch/trikey_gazebo.launch 	modified:   light_ws/src/trikey/trikey_jacobian.py 	new file:   light_ws/src/trikey/urdf/Bumpybot/bumpybot.urdf 	new file:   light_ws/src/trikey/urdf/Bumpybot/bumpybot_simple.urdf 	new file:   light_ws/src/trikey/urdf/Bumpybot/bumpybot_sphere.urdf 	new file:   light_ws/src/trikey/urdf/Bumpybot/meshes/Azure_Kinect.stl 	new file:   light_ws/src/trikey/urdf/Bumpybot/meshes/bumpybot_exterior.stl 	new file:   light_ws/src/trikey/urdf/Bumpybot/meshes/bumpybot_full.stl 	new file:   light_ws/src/trikey/urdf/Bumpybot/meshes/motors_base.stl 	new file:   light_ws/src/trikey/urdf/Bumpybot/meshes/panda.obj 	new file:   light_ws/src/trikey/urdf/Bumpybot/meshes/panda.stl 	new file:   light_ws/src/trikey/urdf/Bumpybot/meshes/panels.mtl 	new file:   light_ws/src/trikey/urdf/Bumpybot/meshes/roller8x750.stl 	new file:   light_ws/src/trikey/urdf/Bumpybot/meshes/rplidar.dae 	new file:   light_ws/src/trikey/urdf/Bumpybot/meshes/teapot.stl 	new file:   light_ws/src/trikey/urdf/Bumpybot/meshes/wheel.stl 	new file:   light_ws/src/trikey/urdf/Bumpybot/trikey.urdf.xacro 	new file:   light_ws/src/trikey/urdf/Bumpybot/trikey_full.urdf 	modified:   light_ws/src/trikey/urdf/trikey_light.urdf.xacro

File: light_ws/src/trikey/urdf/trikey_light.urdf.xacro (robot description, xacro)
@@ -128,5 +128,5 @@
       <child link="wheel_link_${id}"/>
       <axis xyz="0.0 0.0 1.0"/>
-      <limit effort="300.0" velocity="10.0"/>
+      <limit effort="100000000.0" velocity="10.0"/>
     <provideFeedback>true</provideFeedback>
       <physics>
